File: project_venera/project_venera/led_array.kicad_sch (KiCad schematic)
At the start: 36 parts

Commit message: progress on board
Parts:
- LED1, LED10, LED11, LED12, LED13, LED14, LED15, LED16, LED17, LED18, LED19, LED2, LED20, LED21, LED22, LED23, LED24, LED25, LED26, LED27, LED28, LED29, LED3, LED30, LED4, LED5, LED6, LED7, LED8, LED9: footprint SM0603SRC -> LibraryLoader:SM0603SRC
- R10: renamed from R7; value ERJ-PC3B4702V -> TBD; footprint ERJPC3D9763V -> LibraryLoader:ERJPC3D9763V
- R11: renamed from R8; value ERJ-PC3B4702V -> TBD; footprint ERJPC3D9763V -> LibraryLoader:ERJPC3D9763V
- R12: renamed from R9; value ERJ-PC3B4702V -> TBD; footprint ERJPC3D9763V -> LibraryLoader:ERJPC3D9763V
- R7: renamed from R4; value ERJ-PC3B4702V -> TBD; footprint ERJPC3D9763V -> LibraryLoader:ERJPC3D9763V
- R8: renamed from R5; value ERJ-PC3B4702V -> TBD; footprint ERJPC3D9763V -> LibraryLoader:ERJPC3D9763V
- R9: renamed from R6; value ERJ-PC3B4702V -> TBD; footprint ERJPC3D9763V -> LibraryLoader:ERJPC3D9763V
Other:
- note added: "CHARLIEPLEXING ARRAY - 30 LEDS"
- note added: "VENERA LED ARRAY - V1"
- moved on the sheet: LED1, LED10, LED11, LED12, LED14, LED15, LED16, LED17, LED18, LED19, LED2, LED20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

Commit message: update venera hw
Parts:
- renumbered LED11 to LED11_E, LED12 to LED12_R, LED13 to LED13_D, LED14 to LED14_F, LED15 to LED15_X, LED16 to LED16_C, LED18 to LED18_T, LED1 to LED1_Q, LED20 to LED20_Y, LED21 to LED21_G, LED22 to LED22_H, LED23 to LED23_V, LED24 to LED24_B, LED25 to LED25_U, LED26 to LED26_I, LED27 to LED27_J, LED28 to LED28_K, LED29 to LED29_O, LED2 to LED2_A, LED30 to LED30_P, LED3 to LED3_L, LED4 to LED4_N, LED5 to LED5_SPACE, LED6 to LED6_W, LED7 to LED7_S, LED8 to LED8_Z, LED9 to LED9_M
