File: project_venera/project_venera/project_venera.kicad_sch (KiCad schematic)
At the start: 21 parts, among them IC1 NCV303LSN11T1G, IC2 TC1262-3.3VDBTR, IC3 ATSAMD11D14A-SSUT, J1 0022285034, J2 0022285034, J3 0022285034, J4 0022285034, P1 TC2030-CTX

Commit message: progress on board
Parts:
- removed LED_NRST: SM0603SRC, SM0603SRC, symbol LibraryLoader:SM0603SRC
- removed R12: TBD, LibraryLoader:ERJPC3D9763V, symbol LibraryLoader:ERJ-PC3B4702V
- added C3: 100nF, LibraryLoader:C0603, symbol LibraryLoader:C0603C101K5RACAUTO7411
- added S1, S2: B3F-1020, LibraryLoader:B3F1000, symbol LibraryLoader:B3F-1020
- C4: renamed from C3; value 1uF -> 4.7uF
- IC1: footprint SOT95P275X110-5N -> LibraryLoader:SOT95P275X110-5N
- J1, J2: footprint 0022285034 -> LibraryLoader:0022285034
- J3: renamed from J4; footprint 0022285034 -> LibraryLoader:0022285034
- J4: renamed from J3; footprint 0022285034 -> LibraryLoader:0022285034
- LED_REG1: renamed from LED_REG; footprint SM0603SRC -> LibraryLoader:SM0603SRC
- LED_USB1: renamed from LED_USB; footprint SM0603SRC -> LibraryLoader:SM0603SRC
- USB1: footprint Library:USB-C-SMD_GT-USB-7010E-1 -> CustomLib:USB-C-SMD_GT-USB-7010E-1
- renumbered R3 to R1, R1 to R2, R2 to R3, R10 to R4, R11 to R5
Connections:
- net GND: now also C3.1, S1.3, S1.4, S2.3, S2.4
- net KEYBOARD_IN: now also S2.2
- net NRST: now also S1.2
- net VDD: now also C3.2
- no-connect marks 3 -> 7
Other:
- note added: "VENERA MAIN SHEET - V1"
- note removed: "VENERA - V1"
- moved on the sheet: C4, R3

Commit message: update venera hw
Changed lines of the file:
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@@
 		(dnp no)
 		(property "Reference" "R3"
-			(at 58.42 73.6599 90)
+			(at 65.278 73.406 90)
 			(show_name no)
 			(do_not_autoplace no)
@@
 		)
 		(property "Value" "5.1K"
-			(at 58.42 76.1999 90)
+			(at 67.31 76.2 90)
 			(show_name no)
 			(do_not_autoplace no)
